File: RadioModule.kicad_pcb (KiCad board)
At the start: 4 copper layers, 16 x 18 mm, 35 parts, among them J1 Conn_01x01_Pin, J10 Conn_01x01_Pin, J11 Conn_01x01_Pin, J12 Conn_01x01_Pin, J13 Conn_01x01_Pin, J14 Conn_01x01_Pin, J15 Conn_01x01_Pin, J16 Conn_01x01_Pin, J2 Conn_01x01_Pin, J3 Conn_01x01_Pin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

Commit message: Dora the LoRa Module
Parts:
- removed the G*** at (98.5, 77.1)
- added G***: LOGO, LOGO, F.Cu at (101.0, 84.2)
- added G***: LOGO, LOGO, B.Cu at (98.6, 77.6)
Routing:
- net GND: vias 20 -> 18
Other:
- board text added: "Dora The LoRa Module"
- board text added: "SX1280"
- board text removed: "SX1280 Module"
