File: RadioModule.kicad_sch (KiCad schematic)
At the start: 38 parts, among them J1 Conn_01x01_Pin, J10 Conn_01x01_Pin, J11 Conn_01x01_Pin, J12 Conn_01x01_Pin, J13 Conn_01x01_Pin, J14 Conn_01x01_Pin, J15 Conn_01x01_Pin, J16 Conn_01x01_Pin, J2 Conn_01x01_Pin, J3 Conn_01x01_Pin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

Commit message: Crystal Caps sized
Parts:
- C3, C4: value 1nF -> 4pF
Changed lines of the file:
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@@
       (effects (font (size 1.27 1.27)))
     )
-    (property "Value" "1nF" (at 93.98 62.484 0)
+    (property "Value" "4pF" (at 93.98 62.484 0)
       (effects (font (size 1.27 1.27)))
     )
@@
       (effects (font (size 1.27 1.27)))
     )
-    (property "Value" "1nF" (at 93.98 91.694 0)
-      (effects (font (size 1.27 1.27)))
-    )
+    (property "Value" "4pF" (at 93.98 91.694 0)
+      (effects (font (size 1.27 1.27)))
+    )

Commit message: radio module ordering
Parts:
- 3.3VLED1, 3V3LED1: footprint Resistor_SMD:R_0402_1005Metric -> Diode_SMD:D_0402_1005Metric
